File: elc-ludens.cl.kicad_pcb (KiCad board)
At the start: 2 copper layers, 100 x 50 mm, 48 parts, among them P1 CONN_2, P2 CONN_2, P3 CONN_2, P4 CONN_8, Q1 BC337, Q2 BC337, Q3 BC337, Q4 BC337, Q5 BC337, Q6 BC337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

Commit message: Tidy PCB and add Fixing Holes
Must use nylon/plastic hardware to use the fixing holes
Parts:
- added P5: CONN_1, 1pin, F.Cu at (130.0, 142.0)
- added P6: CONN_1, 1pin, F.Cu at (130.0, 98.0)
- added P7: CONN_1, 1pin, F.Cu at (83.0, 118.0)
Routing:
- net GND: track 346.1 -> 569.8 mm
- net /COMP2: track 157.3 -> 160.3 mm
- net N-0000043: track 53.6 -> 52.6 mm
Other:
- board text added: "http://ludens.cl/Electron/picelc/picelc.html"

Commit message: Layout fix BC337 pinout + Add resistor
Parts:
- added R20: 2k2, R5, F.Cu at (77.0, 135.0)
- Q1, Q2, Q3, Q4, Q5, Q6, Q7, Q8: footprint TO92PN -> TO92-EBC
- moved C6 2.50 mm to (80.5, 138.0)
- moved C7 2.50 mm to (80.5, 130.0)
- moved Q1 1.50 mm to (120.0, 137.5)
- moved Q2 1.50 mm to (116.5, 131.0)
- moved Q3 1.50 mm to (120.0, 127.5)
- moved Q4 1.50 mm to (116.5, 121.0)
- moved Q5 1.50 mm to (120.0, 117.5)
- moved Q6 1.50 mm to (116.5, 111.0)
- moved Q7 1.50 mm to (120.0, 107.5)
- moved Q8 1.50 mm to (116.5, 101.0)
- moved X1 1.00 mm to (85.0, 134.0)
Connections:
- net N-0000046 renamed VDD
- R10 pad 1: N-000003 -> N-0000024
- R11 pad 2: N-0000013 -> N-000006
- R12 pad 2: N-0000010 -> N-000002
- R13 pad 2: N-0000034 -> N-0000011
- R14 pad 2: N-0000036 -> N-0000035
- R15 pad 1: N-000009 -> N-000001
- R16 pad 1: N-0000023 -> N-0000015
- R17 pad 1: N-0000033 -> N-0000012
- R18 pad 1: N-0000035 -> N-0000034
- R3 pad 2: N-0000019 -> N-0000029
- R4 pad 2: N-0000016 -> N-0000018
- R5 pad 2: N-000007 -> N-0000027
- R6 pad 2: N-000001 -> N-0000023
- R7 pad 1: N-0000015 -> N-0000022
- R8 pad 1: N-0000020 -> N-0000019
- R9 pad 1: N-000008 -> N-0000028
Routing:
- net GND: track 569.8 -> 519.8 mm
- net N-0000034: track 5.43 -> 24.5 mm
- net N-0000024: track 0.00 -> 11.3 mm
- net N-0000027: track 0.00 -> 8.42 mm
- net N-0000011: track 0.00 -> 8.34 mm
- net N-000006: track 0.00 -> 8.34 mm
- net N-0000029: track 0.00 -> 7.90 mm
- net N-0000022: track 0.00 -> 7.21 mm
- net N-0000020: track 6.89 -> 0.00 mm
- net N-000003: track 6.75 -> 0.00 mm
- net N-0000015: track 4.75 -> 11.0 mm
- net N-0000019: track 5.43 -> 11.3 mm
- net N-0000012: track 0.00 -> 5.65 mm
- net N-0000028: track 0.00 -> 5.65 mm
- net N-000007: track 5.43 -> 0.00 mm
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